File: m2_key_b_3042_template.kicad_pcb (KiCad board)
At the start: 2 copper layers, 42 x 30 mm, 5 parts, among them J1 M.2_Key_B

Commit message: Add note about signal integrity for routing
Other:
- board text added: "Check Table 50. Signal Integrity Parameters For Routing"
Changed lines of the file:
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@@
     (links 72)
     (no_connects 4)
-    (area 84.07143 67.25 166.375 112.000001)
+    (area 84.07143 67.25 166.375 117.625)
     (thickness 1.6)
-    (drawings 23)
+    (drawings 24)
     (tracks 39)
     (zones 0)
@@
       (net 2 GND) (zone_connect 2))
   )
+  (gr_text "Check Table 50. Signal Integrity Parameters\nFor Routing" (at 140 115) (layer Eco1.User)
+    (effects (font (size 1.5 1.5) (thickness 0.3)))
+  )
   (gr_text MAIN (at 158.95 88.4) (layer F.SilkS)
